File: edges/hardware_design/pcb/KiCad/edges_v20_1.kicad_sch (KiCad schematic)
At the start: 50 parts

Commit message: Re-imports
Parts:
- C42, C44: value (none) -> 18p; footprint (none) -> edges_v20:C0603
- C43: value (none) -> 100n; footprint (none) -> edges_v20:C0603
- IC13: value (none) -> MCP3208; footprint (none) -> edges_v20:SO16
- IC15: value (none) -> MCP4822; footprint (none) -> edges_v20:SO08
- IC16: value (none) -> ATXMEGA32A4U-AU; footprint (none) -> edges_v20:TQFP44
- IC5: value (none) -> 741G125DBV; footprint (none) -> edges_v20:SOT23-5
- IC6, IC8: value (none) -> 741G86DBV; footprint (none) -> edges_v20:SOT23-5
- J1, J13, J5, J9: value (none) -> PJ301_THONKICONN6; footprint (none) -> edges_v20:WQP_PJ_301M6
- J18, J20: value (none) -> AVR_SPI_PRG_6PTH; footprint (none) -> edges_v20:2X3
- JP1, JP2, JP3, JP4: value (none) -> FIDUCIAL1X2; footprint (none) -> edges_v20:FIDUCIAL-1X2
- L1: value (none) -> WE-CBF_0603; footprint (none) -> edges_v20:0603
- LED1, LED2, LED3, LED4: value (none) -> LED3MM; footprint (none) -> edges_v20:LED3MM
- Q1, Q2, Q3, Q4: value (none) -> MMBT3904; footprint (none) -> edges_v20:SOT23-BEC
- Q5: value (none) -> 8MHz; footprint (none) -> edges_v20:HC49U70
- R10, R45, R46, R9: value (none) -> 10k; footprint (none) -> edges_v20:R0603
- R20: value (none) -> 1k; footprint (none) -> edges_v20:R0603
- R21, R22, R56, R57: value (none) -> 100k; footprint (none) -> edges_v20:R0603
- R70: value (none) -> 39k; footprint (none) -> edges_v20:R0603
- R71, R72, R73, R74: value (none) -> 100; footprint (none) -> edges_v20:R0603
- SW1, SW2, SW3: value (none) -> S-ON-ONSMALL_SLIDE; footprint (none) -> edges_v20:ES_100SP1T6B11M2QEH_SMALL
- SW4, SW5, SW6, SW7: value (none) -> TAC_SWITCHPTH; footprint (none) -> edges_v20:TACTILE-PTH
