File: edges/hardware_design/pcb/KiCad/edges_v20_2.kicad_sch (KiCad schematic)
At the start: 93 parts

Commit message: Re-imports
Parts:
- C1: value (none) -> 470n; footprint (none) -> edges_v20:C0603
- C10, C12, C23, C26, C29, C31, C4, C6: value (none) -> 100p; footprint (none) -> edges_v20:C0603
- C16, C17: value (none) -> 18p; footprint (none) -> edges_v20:C0603
- C25, C28, C8, C9: value (none) -> 10u; footprint (none) -> edges_v20:PANASONIC_B
- IC10, IC12, IC3, IC4: value (none) -> MCP6002; footprint (none) -> edges_v20:SO08
- IC2, IC7, IC9: value (none) -> TL072D; footprint (none) -> edges_v20:SO08
- J10, J11, J12, J14, J15, J16, J17, J2, J3, J4, J6, J7, J8: value (none) -> PJ301_THONKICONN6; footprint (none) -> edges_v20:WQP_PJ_301M6
- R1: value (none) -> 2k; footprint (none) -> edges_v20:R0603
- R11, R13, R35, R48: value (none) -> 33k; footprint (none) -> edges_v20:R0603
- R12, R17, R23, R44, R47, R52, R58, R8: value (none) -> 24.9k; footprint (none) -> edges_v20:R0603
- R14, R24, R29, R30, R34, R36, R37, R38, R40, R50, R59, R66, R67: value (none) -> 100k; footprint (none) -> edges_v20:R0603
- R15, R18, R2, R53, R60: value (none) -> 10k; footprint (none) -> edges_v20:R0603
- R16, R19, R25, R26, R27, R28, R51, R55, R61, R63, R64, R65: value (none) -> 200k; footprint (none) -> edges_v20:R0603
- R31, R32, R4, R41, R42, R5, R68, R69: value (none) -> 10kB; footprint (none) -> edges_v20:ALPS_POT_VERTICAL_PS
- R33, R43, R49, R6, R7: value (none) -> 1k; footprint (none) -> edges_v20:R0603
- R39: value (none) -> 39k; footprint (none) -> edges_v20:R0603
- R54: value (none) -> 82k; footprint (none) -> edges_v20:R0603
