File: edges/hardware_design/pcb/KiCad/edges_v20_3.kicad_sch (KiCad schematic)
At the start: 46 parts

Commit message: Re-imports
Parts:
- C11, C13, C14, C15, C20, C21, C22, C24, C27, C3, C30, C34, C36, C37, C40, C41, C45, C5, C7: value (none) -> 100n; footprint (none) -> edges_v20:C0603
- C18, C19, C38, C39: value (none) -> 47u; footprint (none) -> edges_v20:PANASONIC_D
- C2, C32: value (none) -> 470n; footprint (none) -> edges_v20:C0603
- C33, C35: value (none) -> 1u; footprint (none) -> edges_v20:C0603
- D1, D2, D3: value (none) -> 1N5819HW; footprint (none) -> edges_v20:SOD123
- IC1: value (none) -> LM4040 10V; footprint (none) -> edges_v20:DBZ_R-PDSO-G3
- IC10, IC12, IC3, IC4: value (none) -> MCP6002; footprint (none) -> edges_v20:SO08
- IC11: value (none) -> LM4040B25; footprint (none) -> edges_v20:DBZ_R-PDSO-G3
- IC14: value (none) -> LM1117-3.3; footprint (none) -> edges_v20:SOT223
- IC2, IC7, IC9: value (none) -> TL072D; footprint (none) -> edges_v20:SO08
- IC5: value (none) -> 741G125DBV; footprint (none) -> edges_v20:SOT23-5
- IC6, IC8: value (none) -> 741G86DBV; footprint (none) -> edges_v20:SOT23-5
- J19: value (none) -> M05X2PTH; footprint (none) -> edges_v20:AVR_ICSP
- R3: value (none) -> 300; footprint (none) -> edges_v20:R0603
- R62: value (none) -> 1k; footprint (none) -> edges_v20:R0603
