File: elements/hardware_design/pcb/KiCad/elements_v02_1.kicad_sch (KiCad schematic)
At the start: 36 parts

Commit message: Re-imports
Parts:
- C11, C12: value (none) -> 18p; footprint (none) -> elements_v02:C0603
- C17, C36, C48: value (none) -> 1u; footprint (none) -> elements_v02:C0603
- C18, C21, C22, C33, C34, C38, C39, C46, C47: value (none) -> 100n; footprint (none) -> elements_v02:C0603
- C31, C35: value (none) -> 2.2u; footprint (none) -> elements_v02:C0805
- C52: value (none) -> 10u; footprint (none) -> elements_v02:PANASONIC_B
- F1, F2, F3, F4: value (none) -> FIDUCIAL1X2; footprint (none) -> elements_v02:FIDUCIAL-1X2
- IC10: value (none) -> STM32F405RGT6; footprint (none) -> elements_v02:TQFP-10X10-64
- IC12: value (none) -> WM8731; footprint (none) -> elements_v02:SSOP28
- JP1: value (none) -> M05X2MINIJTAG; footprint (none) -> elements_v02:2X5-1.27
- JP2: value (none) -> M06SIP; footprint (none) -> elements_v02:1X06
- LED1: value (none) -> SSL-LX5093TC; footprint (none) -> elements_v02:LED5MM
- LED2: value (none) -> SSL-LX5093PC; footprint (none) -> elements_v02:LED5MM
- Q1: value (none) -> 8MHz; footprint (none) -> elements_v02:HC49UP
- R44, R47, R52, R53: value (none) -> 2.2k; footprint (none) -> elements_v02:R0603
- R45, R50: value (none) -> 10k; footprint (none) -> elements_v02:R0603
- SW2, SW3: value (none) -> EVQQ2; footprint (none) -> elements_v02:EVQ-Q2
