File: elements/hardware_design/pcb/KiCad/elements_v02_2.kicad_sch (KiCad schematic)
At the start: 27 parts

Commit message: Re-imports
Parts:
- C40, C53, C55, C56: value (none) -> 10u; footprint (none) -> elements_v02:PANASONIC_B
- C43, C49: value (none) -> 18p; footprint (none) -> elements_v02:C0603
- C44, C45: value (none) -> 100n; footprint (none) -> elements_v02:C0603
- C54, C57: value (none) -> 220p; footprint (none) -> elements_v02:C0603
- IC14: value (none) -> LME49720; footprint (none) -> elements_v02:SO08
- J5, J6, J7, J8: value (none) -> PJ301_THONKICONN6; footprint (none) -> elements_v02:WQP_PJ_301M6
- R51, R59, R69, R72: value (none) -> 47k; footprint (none) -> elements_v02:R0603
- R58, R68, R74, R87: value (none) -> 6.8k; footprint (none) -> elements_v02:R0603
- R75, R86: value (none) -> 36k; footprint (none) -> elements_v02:R0603
- R88, R89: value (none) -> 1.0k; footprint (none) -> elements_v02:R0603
