File: elements/hardware_design/pcb/KiCad/elements_v02_4.kicad_sch (KiCad schematic)
At the start: 42 parts

Commit message: Re-imports
Parts:
- C13, C16, C37, C6: value (none) -> 100n; footprint (none) -> elements_v02:C0603
- IC11, IC3, IC5, IC8: value (none) -> 4051PW; footprint (none) -> elements_v02:TSSOP16
- J3: value (none) -> PJ301_THONKICONN6; footprint (none) -> elements_v02:WQP_PJ_301M6
- Q2: value (none) -> MMBT3904; footprint (none) -> elements_v02:SOT23-BEC
- R10: value (none) -> 33; footprint (none) -> elements_v02:R0603
- R23, R24, R25, R26, R3, R4, R5, R6, R61, R62, R63, R64, R65, R66, R7, R8, R9: value (none) -> 10kB; footprint (none) -> elements_v02:ALPS_POT_VERTICAL_PS
- R60: value (none) -> 10k; footprint (none) -> elements_v02:R0603
- R67: value (none) -> 100k; footprint (none) -> elements_v02:R0603
- R76, R77, R78, R79, R80, R81, R82, R83, R84, R85: value (none) -> 10kB; footprint (none) -> elements_v02:ALPS_POT_VERTICAL
- SW1: value (none) -> LP4OA1PBCT; footprint (none) -> elements_v02:LP4OA1PBCT
- TP1: value (none) -> ADC_TEST; footprint (none) -> elements_v02:PAD.03X.03
