File: elements/hardware_design/pcb/KiCad/elements_v02_5.kicad_sch (KiCad schematic)
At the start: 19 parts

Commit message: Re-imports
Parts:
- C1, C10, C3, C9: value (none) -> 22u; footprint (none) -> elements_v02:PANASONIC_C
- C2, C4, C5, C7, C8: value (none) -> 100n; footprint (none) -> elements_v02:C0603
- D1, D2: value (none) -> 1N5819HW; footprint (none) -> elements_v02:SOD123
- IC1: value (none) -> LM4040B10; footprint (none) -> elements_v02:DBZ_R-PDSO-G3
- IC2, IC4: value (none) -> LM1117-3.3; footprint (none) -> elements_v02:SOT223
- JP3: value (none) -> M05X2PTH; footprint (none) -> elements_v02:AVR_ICSP
- L1, L2: value (none) -> WE-CBF_0603; footprint (none) -> elements_v02:0603
- R1, R2: value (none) -> 1.0k; footprint (none) -> elements_v02:R0603
