File: veils/hardware_design/pcb/KiCad/veils_v40.kicad_pcb (KiCad board)
At the start: 2 copper layers, 59.1 x 106.7 mm, 160 parts, among them IC1 OPA1654, IC10 OPA1654, IC2 LM358PW, IC3 V2164SZ, IC4 OPA1654, IC5 OPA1654, IC6 LM358PW, IC7 V2164SZ, IC8 LM4040C25, IC9 LM4040C10, J1 PJ301_THONKICONN6, J10 PJ301_THONKICONN6, J11 PJ301_THONKICONN6, J12 PJ301_THONKICONN6, J2 PJ301_THONKICONN6, J3 PJ301_THONKICONN6, J4 PJ301_THONKICONN6, J5 PJ301_THONKICONN6, J6 PJ301_THONKICONN6, J7 PJ301_THONKICONN6, J8 PJ301_THONKICONN6, J9 PJ301_THONKICONN6, P1 PTCSMD

Commit message: Re-imports
Connections:
- net Net-(C17-Pad2) renamed OUT2
- net Net-(C26-Pad2) renamed OUT3
- net Net-(C37-Pad2) renamed OUT4
- net Net-(C6-Pad2) renamed OUT1
- net Net-(IC3-Pad2) renamed FOO
- net Net-(IC3-Pad7) renamed FOO1
- net Net-(IC7-Pad2) renamed FOO2
- net Net-(IC7-Pad7) renamed FOO3
- net Net-(J3-PadP3) renamed CV_IN_1
- IC3 pad 1: Net-(IC3-Pad1) -> (no net)
- IC7 pad 1: Net-(IC7-Pad1) -> (no net)
- J11 pad P2: Net-(J11-PadP2) -> (no net)
Other:
- net class Default removed
- rule pad_to_mask_clearance: 0.05 -> 0
- board text added: "Émilie Gillet"
- board text added: "Émilie Gillet,"
