File: ears/hardware_design/pcb/KiCad/ears_v40.kicad_pcb (KiCad board)
At the start: 2 copper layers, 19 x 108.4 mm, 80 parts, among them IC1 OPA1641, IC2 LM324PW, IC3 LM324PW, J1 PJ301_THONKICONN6, J2 PJ301_THONKICONN6, J3 PJ301_THONKICONN6, J4 PJ301_THONKICONN6

Commit message: Redo Ears
Parts:
- removed MIC1: M02TINY, ears_v40:1X02_TINY
- added MIC0: , ears_v40:1X02_TINY, F.Cu at (142.5, 105.6)
- JP1, JP2, JP3: value M03PTH -> (none)
- L1, L2: value WE-CBF_0603 -> (none)
Connections:
- net /ears_v40_2/CLIP renamed CLIP
- net /ears_v40_2/ENVELOPE renamed ENVELOPE
- net /ears_v40_2/FULL_WAVE_RECT renamed FULL_WAVE_RECT
- net /ears_v40_2/GATE renamed GATE
- net /ears_v40_2/~GATE renamed ~{GATE}
- net Net-(C15-Pad2) renamed AMP_OUT_AC
- J2 pad P2: Net-(J2-PadP2) -> (no net)
- J3 pad P2: Net-(J3-PadP2) -> (no net)
- J4 pad P2: Net-(J4-PadP2) -> (no net)
Other:
- net class Default removed
- rule pad_to_mask_clearance: 0.051 -> 0
